Commit message: Commit message

File: dvrk_model/model/gazebo_psm.tool.sca.urdf.xacro (robot description, xacro)
@@ -136,11 +136,11 @@
             <friction>
               <ode>
-                <mu>30.0</mu>
-                <mu2>30.0</mu2>
-              </ode>
-            </friction>
-            <contact>
-              <ode>
-                <kp>1000000.0</kp>
+                <mu>1000.0</mu>
+                <mu2>1000.0</mu2>
+              </ode>
+            </friction>
+            <contact>
+              <ode>
+                <kp>10000.0</kp>
                 <kd>100.0</kd>
                 <max_vel>1.0</max_vel>
@@ -166,4 +166,95 @@
       <origin rpy="0 0 0" xyz="0 0 0"/>
     </joint>
+   <!-- Der-Lin attach fingertip pad 2 blocking block -->
+    <joint name="${prefix}fingertip2_blockjoint" type="fixed">
+      <parent link="${prefix}tool_wrist_sca_ee_link_2"/>
+      <child link="${prefix}tip2_block"/>
+      <axis xyz="0 0 1"/>
+      <origin rpy="0 0 0" xyz="0 0 0"/>
+    </joint>
+  <!-- Der-Lin adding a fingertip2 blocking for grasping -->
+    <link name="${prefix}tip2_block">
+     <visual>
+        <origin rpy="0 0 0" xyz="0.001 0.005 0.0005"/>
+        <geometry>
+          <box size="0.002 0.01 0.004"/>
+        </geometry>
+     </visual>
+      <collision name = "tip2_seg_1">
+        <origin rpy="0 0 0" xyz="0.0 0.010 0.0005"/>
+        <geometry>
+         <cylinder length="0.004" radius="0.0007"/>
+        </geometry>
+       <surface>
+            <friction>
+              <ode>
+                <mu>1000.0</mu>
+                <mu2>1000.0</mu2>
+              </ode>
+            </friction>
+            <contact>
+              <ode>
+                <kp>10000.0</kp>
+                <kd>1000.0</kd>
+                <max_vel>1.0</max_vel>
+                <min_depth>0.001</min_depth>
+              </ode>
+            </contact>
+          </surface>
+      </collision>
+      <collision name = "tip2_seg_2">
+        <origin rpy="0 0 0" xyz="0.0 0.006 0.0005"/>
+        <geometry>
+          <!--box size="0.002 0.001 0.004"/-->
+         <cylinder length="0.004" radius="0.0007"/>
+        </geometry>
+       <surface>
+            <friction>
+              <ode>
+                <mu>1000.0</mu>
+                <mu2>1000.0</mu2>
+              </ode>
+            </friction>
+            <contact>
+              <ode>
+                <kp>10000.0</kp>
+                <kd>1000.0</kd>
+                <max_vel>1.0</max_vel>
+                <min_depth>0.001</min_depth>
+              </ode>
+            </contact>
+          </surface>
+      </collision>
+      <collision name = "tip2_seg_3">
+        <origin rpy="0 0 0.1745" xyz="0.0004 0.008 0.0005"/>
+        <geometry>
+          <box size="0.002 0.002 0.004"/>
+        </geometry>
+       <surface>
+            <friction>
+              <ode>
+                <mu>1000.0</mu>
+                <mu2>1000.0</mu2>
+              </ode>
+            </friction>
+            <contact>
+              <ode>
+                <kp>10000.0</kp>
+                <kd>1000.0</kd>
+                <max_vel>1.0</max_vel>
+                <min_depth>0.001</min_depth>
+              </ode>
+            </contact>
+          </surface>
+      </collision>
+     <inertial>
+      <origin xyz="0 0 0" rpy="0 0 0"/>
+      <mass value="0.05"/>
+      <inertia
+        ixx="0.01" ixy="0.0" ixz="0.0"
+        iyy="0.01" iyz="0.0"
+        izz="0.005"/>
+    </inertial>
+    </link>
 <!-- wsn: other fingertip -->
     <link name="${prefix}fingertip1">
@@ -174,5 +265,5 @@
         </geometry>
      </visual>
-      <collision>
+       <collision>
         <origin rpy="0 0 0" xyz="-0.001 0.005 0.0005"/>
         <geometry>
@@ -182,11 +273,11 @@
             <friction>
               <ode>
-                <mu>30.0</mu>
-                <mu2>30.0</mu2>
-              </ode>
-            </friction>
-            <contact>
-              <ode>
-                <kp>1000000.0</kp>
+                <mu>1000.0</mu>
+                <mu2>1000.0</mu2>
+              </ode>
+            </friction>
+            <contact>
+              <ode>
+                <kp>10000.0</kp>
                 <kd>100.0</kd>
                 <max_vel>1.0</max_vel>
@@ -212,4 +303,96 @@
       <origin rpy="0 0 0" xyz="0 0 0"/>
     </joint>
+    <!-- Der-Lin attach fingertip pad 1 blocking block -->
+    <joint name="${prefix}fingertip1_blockjoint" type="fixed">
+      <parent link="${prefix}tool_wrist_sca_ee_link_1"/>
+      <child link="${prefix}tip1_block"/>
+      <axis xyz="0 0 1"/>
+      <origin rpy="0 0 0" xyz="0 0 0"/>
+    </joint>
+    <!-- Derlin: fingertip1 blocking -->
+    <link name="${prefix}tip1_block">
+     <visual>
+        <origin rpy="0 0 0" xyz="-0.001 0.005 0.0005"/>
+        <geometry>
+          <box size="0.002 0.01 0.004"/>
+        </geometry>
+     </visual>
+       <collision name = "tip1_seg1">
+        <origin rpy="0 0 0" xyz="0.0 0.010 0.0005"/>
+        <geometry>
+          <!--box size="0.003 0.002 0.004"/-->
+          <cylinder length="0.004" radius="0.0007"/>
+        </geometry>
+       <surface>
+            <friction>
+              <ode>
+                <mu>1000.0</mu>
+                <mu2>1000.0</mu2>
+              </ode>
+            </friction>
+            <contact>
+              <ode>
+                <kp>10000.0</kp>
+                <kd>1000.0</kd>
+                <max_vel>1.0</max_vel>
+                <min_depth>0.001</min_depth>
+              </ode>
+            </contact>
+          </surface>
+      </collision>
+      <collision name = "tip1_seg2">
+        <origin rpy="0 0 0" xyz="0.0 0.006 0.0005"/>
+        <geometry>
+          <!--box size="0.002 0.001 0.004"/-->
+         <cylinder length="0.004" radius="0.0007"/>
+        </geometry>
+       <surface>
+            <friction>
+              <ode>
+                <mu>1000.0</mu>
+                <mu2>1000.0</mu2>
+              </ode>
+            </friction>
+            <contact>
+              <ode>
+                <kp>10000.0</kp>
+                <kd>1000.0</kd>
+                <max_vel>1.0</max_vel>
+                <min_depth>0.001</min_depth>
+              </ode>
+            </contact>
+          </surface>
+      </collision>
+     <collision name = "tip1_seg_3">
+        <origin rpy="0 0 -0.1745" xyz="-0.0004 0.008 0.0005"/>
+        <geometry>
+          <box size="0.002 0.002 0.004"/>
+        </geometry>
+       <surface>
+            <friction>
+              <ode>
+                <mu>1000.0</mu>
+                <mu2>1000.0</mu2>
+              </ode>
+            </friction>
+            <contact>
+              <ode>
+                <kp>10000.0</kp>
+                <kd>1000.0</kd>
+                <max_vel>1.0</max_vel>
+                <min_depth>0.001</min_depth>
+              </ode>
+            </contact>
+          </surface>
+      </collision>
+     <inertial>
+      <origin xyz="0 0 0" rpy="0 0 0"/>
+      <mass value="0.05"/>
+      <inertia
+        ixx="0.01" ixy="0.0" ixz="0.0"
+        iyy="0.01" iyz="0.0"
+        izz="0.005"/>
+    </inertial>
+    </link>
     <!-- tool tip -->
     <joint name="${prefix}tool_tip_joint_" type="fixed">

File: dvrk_model/model/gazebo_psm_sticky.tool.sca.urdf.xacro (robot description, xacro)
@@ -136,11 +136,11 @@
             <friction>
               <ode>
-                <mu>3000.0</mu>
-                <mu2>3000.0</mu2>
+                <mu>1000.0</mu>
+                <mu2>1000.0</mu2>
               </ode>
             </friction>
             <contact>
               <ode>
-                <kp>1000000.0</kp>
+                <kp>10000.0</kp>
                 <kd>100.0</kd>
                 <max_vel>1.0</max_vel>
@@ -174,5 +174,5 @@
         </geometry>
      </visual>
-      <collision>
+       <collision>
         <origin rpy="0 0 0" xyz="-0.001 0.005 0.0005"/>
         <geometry>
@@ -182,11 +182,11 @@
             <friction>
               <ode>
-                <mu>3000.0</mu>
-                <mu2>3000.0</mu2>
+                <mu>1000.0</mu>
+                <mu2>1000.0</mu2>
               </ode>
             </friction>
             <contact>
               <ode>
-                <kp>1000000.0</kp>
+                <kp>10000.0</kp>
                 <kd>100.0</kd>
                 <max_vel>1.0</max_vel>
@@ -230,4 +230,23 @@
     <material>Gazebo/Red</material>
   </gazebo>
+<!--Color the sticky fingertips pink, for visibility-->
+		<gazebo reference="${prefix}fingertip1">
+			<material>Gazebo/Purple</material>
+		</gazebo>
+		<!--Create the sticky fingertip.-->
+		<gazebo reference="${prefix}fingertip1">
+			<sensor name="${prefix}fingertip1_sticky" type="contact">
+				<plugin name="${prefix}fingertip1_finger" filename="libsticky_fingers.so">
+					<capacity>25</capacity>
+				</plugin>
+				<contact>
+					<!--For some ungodly reason, the underlying Gazebo touch sensor architecture INSISTS that the name
+					of the contact target be of the form [LINK NAME]_collision. I sincerely wish I was making this up:
+					http://answers.gazebosim.org/question/6929/contact-sensor-error-when-using-gazebo-223/
+					-->
+        	    			<collision>${prefix}fingertip1_collision</collision>
+        	  		</contact>
+       		   	</sensor>
+         	</gazebo>
  <transmission name="${prefix}tran5">
     <type>transmission_interface/SimpleTransmission</type>

File: dvrk_model/model/wsn_both_psms.urdf.xacro (robot description, xacro)
@@ -17,5 +17,5 @@
       <parent link="camera"/>
       <child link="right_camera_link"/>
-      <origin rpy="0.0 1.5708 1.5708" xyz="-0.005 0.0 0.5"/>
+      <origin rpy="0.0 1.5708 1.5708" xyz="-0.0029 0.0 0.5"/>
   </joint>
   <link name="right_camera_link">
@@ -23,5 +23,5 @@
       <origin xyz="0 0 0.0" rpy="0 0 0"/>
       <geometry>
-        <box size="0.03 0.01 0.01"/>
+        <box size="0.02 0.0058 0.0058"/>
       </geometry>
       <material name="red"/>
@@ -37,5 +37,5 @@
       <parent link="camera"/>
       <child link="left_camera_link"/>
-      <origin rpy="0.0 1.5708 1.5708" xyz="0.005 0.00 0.5"/>
+      <origin rpy="0.0 1.5708 1.5708" xyz="0.0029 0.00 0.5"/>
   </joint>
   <link name="left_camera_link">
@@ -43,5 +43,5 @@
       <origin xyz="0 0 0.0" rpy="0 0 0"/>
       <geometry>
-        <box size="0.03 0.01 0.01"/>
+        <box size="0.02 0.0058 0.0058"/>
       </geometry>
       <material name="red"/>
@@ -57,9 +57,11 @@
       prefix="one_"
       parent_link="camera"
-      xyz="-0.15 0.05 0.5" rpy="0.0 0.0 3.1415926"/>
+      xyz="-0.03 0.0 0.5" rpy="0.0 0.0 3.665"/>
+  <!--xyz="-0.15 0.05 0.5" rpy="0.0 0.0 3.1415926"/-->
   <xacro:psm_sca
       prefix="two_"
       parent_link="camera"
-      xyz="0.15 0.05 0.5" rpy="0.0 0.0 3.1415926"/>
+      xyz=" 0.03 0.0 0.5" rpy="0.0 0.0 2.618"/>
+   <!--xyz="0.15 0.05 0.5" rpy="0.0 0.0 3.1415926"/-->
   <!-- ros_control plugin -->
   <gazebo>
@@ -74,5 +76,5 @@
       <update_rate>30.0</update_rate>
       <camera name="right_camera">
-        <horizontal_fov>0.6</horizontal_fov>
+        <horizontal_fov>0.6975</horizontal_fov>
         <image>
           <width>640</width>
@@ -100,5 +102,5 @@
         <cameraInfoTopicName>camera_info</cameraInfoTopicName>
         <frameName>right_camera_link</frameName>
-        <hackBaseline>0.07</hackBaseline>
+        <hackBaseline>-0.0058</hackBaseline>
         <distortionK1>0.0</distortionK1>
         <distortionK2>0.0</distortionK2>
@@ -114,5 +116,5 @@
       <update_rate>30.0</update_rate>
       <camera name="left_camera">
-        <horizontal_fov>0.6</horizontal_fov>
+        <horizontal_fov>0.6975</horizontal_fov>
         <image>
           <width>640</width>
@@ -141,5 +143,5 @@
         <frameName>left_camera_optical_frame</frameName>
         <!--frameName>left_camera_link</frameName-->
-        <hackBaseline>0.07</hackBaseline>
+        <hackBaseline>0.0</hackBaseline>
         <distortionK1>0.0</distortionK1>
         <distortionK2>0.0</distortionK2>

File: dvrk_model/model/wsn_both_psms_rotated_sticky.urdf.xacro (robot description, xacro)
@@ -2,5 +2,5 @@
 <robot name="dvrk_psm" xmlns:xacro="http://www.ros.org/wiki/xacro">
   <!-- Macros -->
-  <xacro:include filename="$(find dvrk_model)/model/wsn_psm.urdf.xacro"/>
+  <xacro:include filename="$(find dvrk_model)/model/wsn_psm_sticky.urdf.xacro"/>
   <link name="world">
       <origin xyz="0.0 0.0 0.0"/>
@@ -70,10 +70,11 @@
       prefix="one_"
       parent_link="camera"
-      xyz="-0.02 0.00 0.50" rpy="0.0 0.0 3.927"/>
+      xyz="-0.08 0.01 0.50" rpy="0.0 0.0 3.141" />
+      <!--xyz="-0.2049 0.0228  0.4527" rpy="-0.0640  -0.02512  3.1347"-->
   <xacro:psm_sca
       prefix="two_"
       parent_link="camera"
-      xyz="0.03 0.00 0.50" rpy="0.0 0.0 2.356"/>
- <!--xyz="0.02 0.00 0.50" rpy="0.0 0.0 2.356"-->
+      xyz="0.08 0.01 0.50" rpy="0.0 0.0 3.141"/>
+      <!-- xyz="0.05 0.01 0.50" rpy="0.0 0.0 2.356" -->
   <!-- ros_control plugin -->
   <gazebo>
